File: Encoder Mount (0.1″ spacing)/Encoder Mount.kicad_pcb (KiCad board)
At the start: 2 copper layers, 23 x 16 mm, 9 parts, among them J1 Conn_01x03_Pin, J2 Conn_01x03_Pin

Commit message: Add version number and tweak alignment
Other:
- board text added: "v1.0"
Changed lines of the file:
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@@
   )
   (footprint "Connector_PinHeader_2.54mm:PinHeader_1x03_P2.54mm_Vertical" (layer "F.Cu")
-    (at 109.91 97.487499)
+    (at 109.91 97.474999)
     (descr "Through hole straight pin header, 1x03, 2.54mm pitch, single row")
     (tags "Through hole pin header THT 1x03 2.54mm single row")
@@
   )
   (footprint "Connector_PinHeader_2.54mm:PinHeader_1x03_P2.54mm_Vertical" (layer "F.Cu")
-    (at 89.59 97.475)
+    (at 89.59 97.474999)
     (descr "Through hole straight pin header, 1x03, 2.54mm pitch, single row")
     (tags "Through hole pin header THT 1x03 2.54mm single row")
@@
     (effects (font (size 0.8 0.8) (thickness 0.15)) (justify top mirror))
   )
+  (gr_text "v1.0" (at 95.300227 105.75 180) (layer "B.SilkS")
+    (effects (font (size 1 1) (thickness 0.15)) (justify mirror))
+  )
   (gr_text "-" (at 108.525001 102.68 180) (layer "B.SilkS")
     (effects (font (size 1 1) (thickness 0.1)))
@@
   (segment (start 89.59 97.475) (end 92.475 97.475) (width 1) (layer "F.Cu") (net 1))
   (segment (start 89.59 102.555) (end 92.445 102.555) (width 1) (layer "F.Cu") (net 2))
-  (segment (start 109.895 100) (end 107.25 100) (width 1) (layer "B.Cu") (net 3))
-  (segment (start 109.91 97.475) (end 107.025 97.475) (width 1) (layer "F.Cu") (net 4))
+  (segment (start 109.895001 100) (end 107.25 100) (width 1) (layer "B.Cu") (net 3))
+  (segment (start 109.91 100.014999) (end 109.895001 100) (width 1) (layer "B.Cu") (net 3))
+  (segment (start 109.91 97.474999) (end 109.909999 97.475) (width 1) (layer "F.Cu") (net 4))
+  (segment (start 109.909999 97.475) (end 107.025 97.475) (width 1) (layer "F.Cu") (net 4))
   (segment (start 107 97.499999) (end 106.350001 97.499999) (width 0.8) (layer "B.Cu") (net 4))
   (segment (start 106.474999 97.499999) (end 104.975 96) (width 0.8) (layer "B.Cu") (net 4))
   (segment (start 106.350001 97.499999) (end 103.85 100) (width 0.8) (layer "B.Cu") (net 4))
-  (segment (start 109.91 102.555) (end 107.055 102.555) (width 1) (layer "F.Cu") (net 5))
+  (segment (start 109.909999 102.555) (end 107.055 102.555) (width 1) (layer "F.Cu") (net 5))
+  (segment (start 109.91 102.554999) (end 109.909999 102.555) (width 1) (layer "F.Cu") (net 5))
   (zone (net 6) (net_name "GND") (layers "F&B.Cu") (hatch edge 0.5)
     (connect_pads yes (clearance 0.5))
