File: Encoder Mount (tight)/Encoder Mount.kicad_pcb (KiCad board)
At the start: 2 copper layers, 20.7 x 15.6 mm, 9 parts, among them J1 Conn_01x03_Pin, J2 Conn_01x03_Pin

Commit message: Add version number and tweak alignment
Other:
- board text added: "v1.0"
Changed lines of the file:
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@@
   )
   (footprint "Connector_PinHeader_2.54mm:PinHeader_1x03_P2.54mm_Vertical" (layer "F.Cu")
-    (at 109.04 97.487499)
+    (at 109.04 97.474999)
     (descr "Through hole straight pin header, 1x03, 2.54mm pitch, single row")
     (tags "Through hole pin header THT 1x03 2.54mm single row")
@@
   )
   (footprint "Connector_PinHeader_2.54mm:PinHeader_1x03_P2.54mm_Vertical" (layer "F.Cu")
-    (at 90.46 97.475)
+    (at 90.46 97.474999)
     (descr "Through hole straight pin header, 1x03, 2.54mm pitch, single row")
     (tags "Through hole pin header THT 1x03 2.54mm single row")
@@
     (effects (font (size 1 1) (thickness 0.15)) (justify bottom mirror))
   )
+  (gr_text "v1.0" (at 95.610894 105.75 180) (layer "B.SilkS")
+    (effects (font (size 1 1) (thickness 0.15)) (justify mirror))
+  )
   (gr_text "G→2" (at 102.10381 93.5 180) (layer "B.SilkS")
     (effects (font (size 0.8 0.8) (thickness 0.15)) (justify left bottom mirror))
@@
   (segment (start 90.46 97.475) (end 92.475 97.475) (width 1) (layer "F.Cu") (net 1))
   (segment (start 90.46 102.555) (end 92.445 102.555) (width 1) (layer "F.Cu") (net 2))
-  (segment (start 109.04 100.027499) (end 107 100.027499) (width 1) (layer "B.Cu") (net 3))
-  (segment (start 107 97.499999) (end 109.0275 97.499999) (width 1) (layer "F.Cu") (net 4))
+  (segment (start 109.0275 100.027499) (end 107 100.027499) (width 1) (layer "B.Cu") (net 3))
+  (segment (start 107 97.499999) (end 109.015 97.499999) (width 1) (layer "F.Cu") (net 4))
   (segment (start 103.35 100) (end 105.850001 97.499999) (width 0.8) (layer "B.Cu") (net 4))
   (segment (start 105.999999 97.499999) (end 104.5 96) (width 0.8) (layer "B.Cu") (net 4))
   (segment (start 105.850001 97.499999) (end 107 97.499999) (width 0.8) (layer "B.Cu") (net 4))
   (segment (start 107 97.499999) (end 105.999999 97.499999) (width 0.8) (layer "B.Cu") (net 4))
-  (segment (start 109.04 102.567499) (end 107.0675 102.567499) (width 1) (layer "F.Cu") (net 5))
+  (segment (start 109.04 102.554999) (end 107.055 102.554999) (width 1) (layer "F.Cu") (net 5))
   (zone (net 6) (net_name "GND") (layers "F&B.Cu") (hatch edge 0.5)
     (connect_pads yes (clearance 0.25))
