File: Encoder Mount (tight)/Encoder Mount.kicad_pcb (KiCad board)
At the start: 2 copper layers, 20.7 x 15.6 mm, 9 parts, among them J1 Conn_01x03_Pin, J2 Conn_01x03_Pin

Commit message: Add JLC order number locator
See [“ How to remove order number from your PCB?”](https://jlcpcb.com/help/article/50-How-to-remove-order-number-from-your-PCB)
Other:
- board text added: "JLCJLCJLCJLC"
Changed lines of the file:
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@@
     (effects (font (size 0.8 0.8) (thickness 0.15)) (justify bottom))
+  )
+  (gr_text "JLCJLCJLCJLC" (at 96 99.999999 90) (layer "F.SilkS")
+    (effects (font (size 0.8 0.8) (thickness 0.15)))
   )
   (gr_text "-" (at 105.45 102.4025) (layer "F.SilkS")
